File: power.brd (EAGLE design)
At the start: 50 x 25 mm, 21 parts, among them CON1 4UCON-19963, CON2 4UCON-19836, CON3 4UCON-10709, CON4 4UCON-10709, IC1 TPS62133, SW1 SWITCHSWITCH

Commit message: Final update for version 2
Routing:
- net VCC: track 80.3 -> 78.6 mm
- net SS/TR: track 11.2 -> 10.4 mm
Other:
- board text added: "2014-07-25"
- board text removed: "2014-02-23"
Changed lines of the file:
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@@
 <setting verticaltext="up"/>
 </settings>
-<grid distance="1" unitdist="mm" unit="mm" style="lines" multiple="1" display="yes" altdistance="0.5" altunitdist="mm" altunit="mm"/>
+<grid distance="1" unitdist="mm" unit="mm" style="lines" multiple="1" display="yes" altdistance="0.1" altunitdist="mm" altunit="mm"/>
 <layers>
 <layer number="1" name="Top" color="4" fill="1" visible="yes" active="yes"/>
@@
 <layer number="220" name="220bmp" color="21" fill="1" visible="no" active="no"/>
 <layer number="221" name="221bmp" color="22" fill="1" visible="no" active="no"/>
-<layer number="222" name="222bmp" color="23" fill="1" visible="no" active="no"/>
 <layer number="223" name="223bmp" color="24" fill="1" visible="no" active="no"/>
 <layer number="224" name="224bmp" color="25" fill="1" visible="no" active="no"/>
@@
 <text x="0" y="-3" size="1.778" layer="48" font="vector" ratio="12">Power Board</text>
 <text x="50" y="-3" size="1.778" layer="48" font="vector" ratio="12" align="bottom-right">Version: 2</text>
-<text x="50" y="-6" size="1.27" layer="48" font="vector" ratio="12" align="bottom-right">2014-02-23</text>
+<text x="50" y="-6" size="1.27" layer="48" font="vector" ratio="12" align="bottom-right">2014-07-25</text>
 <text x="0" y="-6" size="1.27" layer="48" font="vector" ratio="12">http://robopoly.epfl.ch</text>
 <text x="0" y="-9" size="1.27" layer="48" font="vector" ratio="12">Licence: Creative Commons</text>
@@
 <contactref element="SW1" pad="1"/>
 <contactref element="JP1" pad="2"/>
-<wire x1="25.75" y1="14.6" x2="26.3" y2="14.7" width="0.3048" layer="1"/>
-<wire x1="26.3" y1="14.7" x2="26.7" y2="14.3" width="0.3048" layer="1"/>
-<wire x1="26.7" y1="14.3" x2="26.6" y2="13.75" width="0.3048" layer="1"/>
 <wire x1="26.6" y1="13.75" x2="26.6" y2="13.25" width="0.3048" layer="1"/>
 <wire x1="26.6" y1="13.25" x2="26.6" y2="12.75" width="0.3048" layer="1"/>
@@
 <vertex x="26" y="14"/>
 <vertex x="26" y="12.5"/>
-<vertex x="27" y="12.5"/>
-<vertex x="27" y="13.5"/>
+<vertex x="26.75" y="12.5"/>
+<vertex x="27.75" y="13.5"/>
 <vertex x="29.5" y="13.5"/>
-<vertex x="29.5" y="14.5"/>
-<vertex x="26.5" y="14.5"/>
+<vertex x="29.5" y="14.4"/>
+<vertex x="26.6" y="14.4"/>
 <vertex x="26" y="15"/>
 </polygon>
@@
 <via x="28" y="12.25" extent="1-16" drill="0.6" shape="octagon"/>
 <via x="20" y="12.05" extent="1-16" drill="0.6" shape="octagon"/>
-<wire x1="20" y1="12.05" x2="22.05" y2="10" width="0.3048" layer="16"/>
-<wire x1="22.05" y1="10" x2="25.75" y2="10" width="0.3048" layer="16"/>
-<wire x1="25.75" y1="10" x2="28" y2="12.25" width="0.3048" layer="16"/>
+<wire x1="20" y1="12.05" x2="21.05" y2="11" width="0.3048" layer="16"/>
+<wire x1="21.05" y1="11" x2="26.75" y2="11" width="0.3048" layer="16"/>
+<wire x1="26.75" y1="11" x2="28" y2="12.25" width="0.3048" layer="16"/>
 </signal>
 <signal name="5V/3A">
